File: battery-pack-pcb/_autosave-battery-pack-pcb.sch (KiCad schematic (older format))
At the start: 7 parts, among them J1 Conn_01x02_Female, J2 Conn_01x02_Female

Commit message: Add capacitor to battery pack
Parts:
- added C1: C_Small, Capacitor_SMD:C_1210_3225Metric_Pad1.42x2.65mm_HandSolder, symbol Device:C_Small
- D1, D2: symbol Device:D_Small -> Device:D_Schottky_Small
Connections:
- wire segments 26 -> 30
Changed lines of the file:
@@
 $EndComp
 $Comp
-L Device:D_Small D1
+L Device:D_Schottky_Small D1
 U 1 1 5D5C10F0
 P 3500 2500
@@
 $EndComp
 $Comp
-L Device:D_Small D2
+L Device:D_Schottky_Small D2
 U 1 1 5D5C26DF
 P 4400 2500
@@
 	3750 3550 3750 3950
 Wire Wire Line
-	3750 3950 5250 3950
+	3750 3950 4900 3950
 Connection ~ 3750 3550
 Wire Wire Line
@@
 $EndComp
 Wire Wire Line
-	4600 1950 5300 1950
+	4600 1950 4900 1950
 Wire Wire Line
 	5300 1950 5300 2050
@@
 Wire Wire Line
 	4500 2500 4600 2500
+$Comp
+L Device:C_Small C1
+U 1 1 5D987608
+P 4900 2500
+F 0 "C1" H 4992 2546 50  0000 L CNN
+F 1 "C_Small" H 4992 2455 50  0000 L CNN
+F 2 "Capacitor_SMD:C_1210_3225Metric_Pad1.42x2.65mm_HandSolder" H 4900 2500 50  0001 C CNN
+F 3 "~" H 4900 2500 50  0001 C CNN
+	1    4900 2500
+	1    0    0    -1
+$EndComp
+Wire Wire Line
+	4900 1950 4900 2400
+Connection ~ 4900 1950
+Wire Wire Line
+	4900 1950 5300 1950
+Wire Wire Line
+	4900 2600 4900 3950
+Connection ~ 4900 3950
+Wire Wire Line
+	4900 3950 5250 3950
 $EndSCHEMATC
