File: _autosave-caravelle.sch (KiCad schematic (older format))
At the start: 71 parts, among them J1 Conn_01x04, J2 Conn_01x02_Female, J3 Conn_01x04, J4 Conn_01x02_Female, J5 Conn_01x01, J6 Conn_01x01, K1 keyboard_parts_KEYSW, K10 keyboard_parts_KEYSW, K11 keyboard_parts_KEYSW, K12 keyboard_parts_KEYSW, K13 keyboard_parts_KEYSW, K14 keyboard_parts_KEYSW, K15 keyboard_parts_KEYSW, K16 keyboard_parts_KEYSW, K17 keyboard_parts_KEYSW, K18 keyboard_parts_KEYSW, K19 keyboard_parts_KEYSW, K2 keyboard_parts_KEYSW, K20 keyboard_parts_KEYSW, K21 keyboard_parts_KEYSW, K22 keyboard_parts_KEYSW, K23 keyboard_parts_KEYSW, K24 keyboard_parts_KEYSW, K25 keyboard_parts_KEYSW, K26 keyboard_parts_KEYSW, K27 keyboard_parts_KEYSW, K28 keyboard_parts_KEYSW, K29 keyboard_parts_KEYSW, K3 keyboard_parts_KEYSW, K30 keyboard_parts_KEYSW, K31 keyboard_parts_KEYSW, K32 keyboard_parts_KEYSW, K33 keyboard_parts_KEYSW, K34 keyboard_parts_KEYSW, K35 keyboard_parts_KEYSW, K36 keyboard_parts_KEYSW, K37 keyboard_parts_KEYSW, K38 keyboard_parts_KEYSW, K39 keyboard_parts_KEYSW, K4 keyboard_parts_KEYSW, K40 keyboard_parts_KEYSW, K41 keyboard_parts_KEYSW, K42 keyboard_parts_KEYSW, K43 keyboard_parts_KEYSW, K44 keyboard_parts_KEYSW, K45 keyboard_parts_KEYSW, K46 keyboard_parts_KEYSW, K47 keyboard_parts_KEYSW, K48 keyboard_parts_KEYSW, K5 keyboard_parts_KEYSW, K6 keyboard_parts_KEYSW, K7 keyboard_parts_KEYSW, K8 keyboard_parts_KEYSW, K9 keyboard_parts_KEYSW, SW1 SW_SPDT, SW2 SW_SPDT, SW3 RESET_SW, SW4 RESET_SW, U1 BL652_LEFT, U11 logo1, U12 logo2, U13 logo1, U2 hole, U3 hole, U4 hole, U5 BL652_RIGHT, U6 hole, U7 hole, U8 hole

Commit message: Add DFU button
Parts:
- J5, J6: footprint Jumper:SolderJumper-2_P1.3mm_Bridged2Bar_Pad1.0x1.5mm -> locallib:breakout-pad
Changed lines of the file:
@@
 F 0 "J5" H 4030 3142 50  0000 L CNN
 F 1 "Conn_01x01" H 4030 3051 50  0000 L CNN
-F 2 "Jumper:SolderJumper-2_P1.3mm_Bridged2Bar_Pad1.0x1.5mm" H 3950 3100 50  0001 C CNN
+F 2 "locallib:breakout-pad" H 3950 3100 50  0001 C CNN
 F 3 "~" H 3950 3100 50  0001 C CNN
 	1    3950 3100
@@
 F 0 "J6" H 4080 7342 50  0000 L CNN
 F 1 "Conn_01x01" H 4080 7251 50  0000 L CNN
-F 2 "Jumper:SolderJumper-2_P1.3mm_Bridged2Bar_Pad1.0x1.5mm" H 4000 7300 50  0001 C CNN
+F 2 "locallib:breakout-pad" H 4000 7300 50  0001 C CNN
 F 3 "~" H 4000 7300 50  0001 C CNN
 	1    4000 7300
