File: caravelle.kicad_pcb (KiCad board)
At the start: 2 copper layers, 277.4 x 94.1 mm, 83 parts, among them J1 Conn_01x04, J2 Conn_01x02_Female, J3 Conn_01x04, J4 Conn_01x02_Female, K1 keyboard_parts_KEYSW, K10 keyboard_parts_KEYSW, K11 keyboard_parts_KEYSW, K12 keyboard_parts_KEYSW, K13 keyboard_parts_KEYSW, K14 keyboard_parts_KEYSW, K15 keyboard_parts_KEYSW, K16 keyboard_parts_KEYSW, K17 keyboard_parts_KEYSW, K18 keyboard_parts_KEYSW, K19 keyboard_parts_KEYSW, K2 keyboard_parts_KEYSW, K20 keyboard_parts_KEYSW, K21 keyboard_parts_KEYSW, K22 keyboard_parts_KEYSW, K23 keyboard_parts_KEYSW, K24 keyboard_parts_KEYSW, K25 keyboard_parts_KEYSW, K26 keyboard_parts_KEYSW, K27 keyboard_parts_KEYSW, K28 keyboard_parts_KEYSW, K29 keyboard_parts_KEYSW, K3 keyboard_parts_KEYSW, K30 keyboard_parts_KEYSW, K31 keyboard_parts_KEYSW, K32 keyboard_parts_KEYSW, K33 keyboard_parts_KEYSW, K34 keyboard_parts_KEYSW, K35 keyboard_parts_KEYSW, K36 keyboard_parts_KEYSW, K37 keyboard_parts_KEYSW, K38 keyboard_parts_KEYSW, K39 keyboard_parts_KEYSW, K4 keyboard_parts_KEYSW, K40 keyboard_parts_KEYSW, K41 keyboard_parts_KEYSW, K42 keyboard_parts_KEYSW, K43 keyboard_parts_KEYSW, K44 keyboard_parts_KEYSW, K45 keyboard_parts_KEYSW, K46 keyboard_parts_KEYSW, K47 keyboard_parts_KEYSW, K48 keyboard_parts_KEYSW, K5 keyboard_parts_KEYSW, K6 keyboard_parts_KEYSW, K7 keyboard_parts_KEYSW, K8 keyboard_parts_KEYSW, K9 keyboard_parts_KEYSW, SW1 SW_SPDT, SW2 SW_SPDT, U1 MDBT40_LEFT, U10 STLQ015M33R, U11 logo1, U12 logo2, U13 logo1, U2 hole, U3 hole, U4 hole, U5 MDBT40_RIGHT, U6 hole, U7 hole, U8 hole, U9 STLQ015M33R, Y1 32.768kHz, Y2 32.768kHz

Commit message: Add v2.0 PCB
Parts:
- removed C2, C3, C5, C6: 12pF, Capacitor_SMD:C_0603_1608Metric_Pad1.05x0.95mm_HandSolder
- removed Y1, Y2: 32.768kHz, Crystal:Crystal_SMD_3215-2Pin_3.2x1.5mm
- added R1: R_Small, Resistor_SMD:R_0603_1608Metric_Pad1.05x0.95mm_HandSolder, F.Cu at (58.8, 120.4)
- added R2: R_Small, Resistor_SMD:R_0603_1608Metric_Pad1.05x0.95mm_HandSolder, F.Cu at (318.6, 120.4)
- added SW3: RESET_SW, locallib:SW_SPST_ALPS-SKRP, F.Cu at (55.3, 116.2)
- added SW4: RESET_SW, locallib:SW_SPST_ALPS-SKRP, F.Cu at (322.1, 116.2)
- C1, C4: value 1uF -> 0.1uF
- U1: value MDBT40_LEFT -> BL652_LEFT; footprint locallib:MDBT40 -> RF_Module:Laird_BL652
- U5: value MDBT40_RIGHT -> BL652_RIGHT; footprint locallib:MDBT40 -> RF_Module:Laird_BL652
- moved J3 50.4 mm to (306.4, 127.8), turned to 180 degrees
- moved J1 43.6 mm to (71.0, 127.8), turned to 180 degrees
- moved D2 26.2 mm to (67.2, 126.4), turned to 270 degrees
- moved D4 25.5 mm to (310.2, 126.4), turned to 270 degrees
- moved C1 17.2 mm to (86.2, 113.8), turned to 0 degrees
- moved C4 12.9 mm to (299.6, 113.8), turned to 0 degrees
- moved SW2 3.98 mm to (310.9, 117.3)
- moved SW1 3.98 mm to (60.5, 117.3)
- moved C9 3.15 mm to (316.4, 120.4)
- moved U10 2.75 mm to (313.0, 120.4)
- moved J4 2.71 mm to (313.9, 127.2)
- moved C10 2.45 mm to (309.6, 120.4)
- moved U12 2.10 mm to (80.4, 76.6)
- moved J2 1.68 mm to (63.5, 125.2)
- moved D1 1.66 mm to (56.4, 120.8), turned to 270 degrees
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Connections:
- U1 pad 10: /XL1 -> /L1
- U1 pad 11: Net-(U1-Pad11) -> /L15
- U1 pad 12: Net-(U1-Pad12) -> /L8
- U1 pad 13: GND -> /L2
- U1 pad 14: VCC -> Net-(U1-Pad14)
- U1 pad 16: /L17 -> GND
- U1 pad 17: /L10 -> /L16
- U1 pad 18: /L4 -> /L9
- U1 pad 19: /L15 -> /L3
- U1 pad 2: GND -> Net-(U1-Pad2)
- U1 pad 20: /L8 -> /L17
- U1 pad 21: /L2 -> /L10
- U1 pad 22: /L1 -> /L4
- U1 pad 23: /L7 -> /L18
- U1 pad 24: /L14 -> Net-(U1-Pad24)
- U1 pad 25: GND -> Net-(U1-Pad25)
- U1 pad 26: Net-(U1-Pad26) -> VCC
- U1 pad 27: /L20 -> GND
- U1 pad 28: /L13 -> /L11
- U1 pad 29: /L6 -> /L5
- U1 pad 3: VCC -> Net-(U1-Pad3)
- U1 pad 30: /L18 -> /L19
- U1 pad 31: /L11 -> /L12
- U1 pad 32: /L5 -> /L6
- U1 pad 33: /L19 -> /L13
- U1 pad 34: /L12 -> /L20
- U1 pad 35: /SWDIO -> /L21
- U1 pad 36: /SWDCLK -> /L22
- U1 pad 37: /L21 -> /L23
- U1 pad 38: /L22 -> /L24
- U1 pad 39: /L23 -> GND
- U1 pad 5: /L16 -> /SWDIO
- U1 pad 6: /L9 -> /SWDCLK
- U1 pad 7: /L3 -> Net-(SW3-Pad1)
- U1 pad 8: Net-(U1-Pad8) -> /L14
- U1 pad 9: /XL2 -> /L7
- U5 pad 10: /XL1_R -> /R13
- U5 pad 11: Net-(U5-Pad11) -> /R19
- U5 pad 12: Net-(U5-Pad12) -> /R12
- U5 pad 13: GNDA -> /R6
- U5 pad 14: VAA -> /R18
- U5 pad 15: Net-(U5-Pad15) -> /R11
- U5 pad 16: /R14 -> GNDA
- U5 pad 17: /R7 -> /R5
- U5 pad 18: /R1 -> /R17
- U5 pad 19: /R2 -> /R10
- U5 pad 2: GNDA -> /R24
- U5 pad 20: /R8 -> /R4
- U5 pad 21: /R15 -> /R16
- U5 pad 22: /R20 -> /R9
- U5 pad 23: /R13 -> /R3
- U5 pad 24: /R19 -> Net-(U5-Pad24)
- U5 pad 25: GNDA -> Net-(U5-Pad25)
- U5 pad 26: Net-(U5-Pad26) -> VAA
- U5 pad 27: /R3 -> GNDA
- U5 pad 28: /R9 -> /R15
- U5 pad 29: /R16 -> /R8
- U5 pad 3: VAA -> /R23
- U5 pad 30: /R4 -> /R2
- U5 pad 31: /R10 -> /R1
- U5 pad 32: /R17 -> /R7
- U5 pad 33: /R5 -> /R14
- U5 pad 34: /R11 -> Net-(U5-Pad34)
- U5 pad 35: /SWDIO_R -> Net-(U5-Pad35)
- U5 pad 36: /SWDCLK_R -> Net-(U5-Pad36)
- U5 pad 37: /R18 -> Net-(U5-Pad37)
- U5 pad 38: /R6 -> Net-(U5-Pad38)
- U5 pad 39: /R12 -> GNDA
- U5 pad 4: /R21 -> /R22
- U5 pad 5: /R22 -> /SWDIO_R
- U5 pad 6: /R23 -> /SWDCLK_R
- U5 pad 7: /R24 -> Net-(SW4-Pad1)
- U5 pad 8: Net-(U5-Pad8) -> /R21
- U5 pad 9: /XL2_R -> /R20
Routing:
- net Net-(SW4-Pad1): track 0.00 -> 48.6 mm, vias 0 -> 2
- net /SWDCLK: track 46.1 -> 7.58 mm
- net /SWDIO: track 43.4 -> 6.73 mm
- net Net-(SW3-Pad1): track 0.00 -> 30.8 mm, vias 0 -> 2
- net Net-(D4-Pad2): track 30.7 -> 3.90 mm
- net /SWDIO_R: track 38.2 -> 16.6 mm, vias 0 -> 1
- net /L21: track 38.9 -> 19.6 mm
- net /L2: track 85.2 -> 66.6 mm, vias 2 -> 0
- net /L20: track 130.5 -> 113.0 mm, vias 2 -> 0
- net /L13: track 148.8 -> 131.4 mm, vias 2 -> 0
- net /SWDCLK_R: track 34.6 -> 17.4 mm, vias 0 -> 1
- net /L6: track 148.2 -> 131.0 mm, vias 2 -> 0
- net Net-(D2-Pad2): track 20.5 -> 3.90 mm
- net /R21: track 29.5 -> 13.4 mm, vias 2 -> 0
- net /VCC_BAT_R: track 39.8 -> 23.8 mm, vias 0 -> 1
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- removed copper zone on F.Cu, net GND
- removed copper zone on F.Cu, net GNDA
Other:
- outline, holes or cut-outs redrawn
- board text added: "Caravelle-BLE PCB v2.0 by SatT"
- board text removed: "Caravelle PCB v1.5 by SatT"

Commit message: Minor fix to routing
Routing:
- net /R5: track 93.9 -> 94.5 mm
Changed lines of the file:
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@@
     (thickness 1.6)
     (drawings 118)
-    (tracks 584)
+    (tracks 586)
     (zones 0)
     (modules 81)
@@
   (segment (start 292.918446 112.799946) (end 290.281554 112.799946) (width 0.2) (layer F.Cu) (net 37))
   (segment (start 290.281554 112.799946) (end 290.281531 112.799969) (width 0.2) (layer F.Cu) (net 37))
+  (segment (start 293.85 114.95) (end 293.85 115.7) (width 0.2) (layer F.Cu) (net 38))
   (segment (start 292.9 114) (end 293.85 114.95) (width 0.2) (layer F.Cu) (net 38))
   (segment (start 290.778598 114) (end 290.778621 113.999977) (width 0.2) (layer F.Cu) (net 38))
   (segment (start 284.589455 110.766757) (end 287.822698 114) (width 0.2) (layer F.Cu) (net 38))
-  (segment (start 290.778621 113.999977) (end 292.421379 113.999977) (width 0.2) (layer F.Cu) (net 38))
-  (segment (start 287.822698 114) (end 290.778598 114) (width 0.2) (layer F.Cu) (net 38) (status 40000))
-  (segment (start 263.825 55.025) (end 270 61.2) (width 0.2) (layer F.Cu) (net 38))
-  (segment (start 263.225 55.025) (end 263.825 55.025) (width 0.2) (layer F.Cu) (net 38))
-  (segment (start 270 61.2) (end 270 105.3) (width 0.2) (layer F.Cu) (net 38))
-  (segment (start 292.421379 113.999977) (end 292.421402 114) (width 0.2) (layer F.Cu) (net 38))
   (segment (start 284.566757 110.766757) (end 284.589455 110.766757) (width 0.2) (layer F.Cu) (net 38))
-  (segment (start 270 105.3) (end 270.323224 105.623224) (width 0.2) (layer F.Cu) (net 38))
-  (segment (start 270.323224 105.623224) (end 279.423224 105.623224) (width 0.2) (layer F.Cu) (net 38))
-  (segment (start 293.85 114.95) (end 293.85 115.7) (width 0.2) (layer F.Cu) (net 38))
+  (segment (start 279.499978 105.699979) (end 284.566757 110.766757) (width 0.2) (layer F.Cu) (net 38))
+  (segment (start 270.399904 105.699904) (end 273.131296 105.699906) (width 0.2) (layer F.Cu) (net 38))
   (segment (start 292.421402 114) (end 292.9 114) (width 0.2) (layer F.Cu) (net 38))
-  (segment (start 279.423224 105.623224) (end 284.566757 110.766757) (width 0.2) (layer F.Cu) (net 38))
-  (segment (start 272.634306 106.900011) (end 279.002911 106.900011) (width 0.2) (layer F.Cu) (net 39))
-  (segment (start 284.092388 111.96679) (end 287.625598 115.5) (width 0.2) (layer F.Cu) (net 39))
-  (segment (start 279.002911 106.900011) (end 284.06969 111.96679) (width 0.2) (layer F.Cu) (net 39))
-  (segment (start 251 105.454937) (end 252.44499 106.899927) (width 0.2) (layer F.Cu) (net 39))
-  (segment (start 284.06969 111.96679) (end 284.092388 111.96679) (width 0.2) (layer F.Cu) (net 39))
+  (segment (start 270 105.3) (end 270.399904 105.699904) (width 0.2) (layer F.Cu) (net 38))
+  (segment (start 292.421379 113.999977) (end 292.421402 114) (width 0.2) (layer F.Cu) (net 38))
+  (segment (start 270 61.2) (end 270 105.3) (width 0.2) (layer F.Cu) (net 38))
+  (segment (start 263.825 55.025) (end 270 61.2) (width 0.2) (layer F.Cu) (net 38))
+  (segment (start 273.131296 105.699906) (end 273.131369 105.699979) (width 0.2) (layer F.Cu) (net 38))
+  (segment (start 263.225 55.025) (end 263.825 55.025) (width 0.2) (layer F.Cu) (net 38))
+  (segment (start 287.822698 114) (end 290.778598 114) (width 0.2) (layer F.Cu) (net 38))
+  (segment (start 290.778621 113.999977) (end 292.421379 113.999977) (width 0.2) (layer F.Cu) (net 38))
+  (segment (start 273.131369 105.699979) (end 279.499978 105.699979) (width 0.2) (layer F.Cu) (net 38))
   (segment (start 291.4 115.5) (end 291.6 115.7) (width 0.2) (layer F.Cu) (net 39))
+  (segment (start 284.06969 111.96679) (end 284.092388 111.96679) (width 0.2) (layer F.Cu) (net 39))
+  (segment (start 279.002911 106.900011) (end 284.06969 111.96679) (width 0.2) (layer F.Cu) (net 39))
+  (segment (start 272.634306 106.900011) (end 279.002911 106.900011) (width 0.2) (layer F.Cu) (net 39))
+  (segment (start 251 65.992499) (end 251 106.5) (width 0.2) (layer F.Cu) (net 39))
+  (segment (start 287.625598 115.5) (end 291.4 115.5) (width 0.2) (layer F.Cu) (net 39))
   (segment (start 244.215 59.207499) (end 251 65.992499) (width 0.2) (layer F.Cu) (net 39))
-  (segment (start 272.634229 106.899934) (end 272.634306 106.900011) (width 0.2) (layer F.Cu) (net 39))
+  (segment (start 251 106.5) (end 251.399928 106.899928) (width 0.2) (layer F.Cu) (net 39))
+  (segment (start 251.399928 106.899928) (end 253.244211 106.899928) (width 0.2) (layer F.Cu) (net 39))
   (segment (start 253.244211 106.899928) (end 272.634229 106.899934) (width 0.2) (layer F.Cu) (net 39))
-  (segment (start 252.44499 106.899927) (end 253.244211 106.899928) (width 0.2) (layer F.Cu) (net 39))
-  (segment (start 251 65.992499) (end 251 105.454937) (width 0.2) (layer F.Cu) (net 39))
-  (segment (start 287.625598 115.5) (end 291.4 115.5) (width 0.2) (layer F.Cu) (net 39))
+  (segment (start 284.092388 111.96679) (end 287.625598 115.5) (width 0.2) (layer F.Cu) (net 39))
+  (segment (start 272.634229 106.899934) (end 272.634306 106.900011) (width 0.2) (layer F.Cu) (net 39))
   (segment (start 289.65 118.4) (end 290.45 118.4) (width 0.2) (layer F.Cu) (net 40))
   (segment (start 272.137156 108.099961) (end 272.137239 108.100044) (width 0.2) (layer F.Cu) (net 40))
@@
   (segment (start 282.846875 77.646875) (end 282.275 77.646875) (width 0.2) (layer F.Cu) (net 43))
   (segment (start 290.447243 113.199957) (end 290.44722 113.19998) (width 0.2) (layer F.Cu) (net 43))
-  (segment (start 279.334289 106.099989) (end 284.401068 111.166768) (width 0.2) (layer F.Cu) (net 44))
   (segment (start 284.423766 111.166768) (end 287.657009 114.400011) (width 0.2) (layer F.Cu) (net 44))
-  (segment (start 290.94431 114.399988) (end 292.25569 114.399988) (width 0.2) (layer F.Cu) (net 44))
-  (segment (start 292.25569 114.399988) (end 292.255713 114.400011) (width 0.2) (layer F.Cu) (net 44))
-  (segment (start 292.600011 114.400011) (end 293.1 114.9) (width 0.2) (layer F.Cu) (net 44))
-  (segment (start 292.255713 114.400011) (end 292.600011 114.400011) (width 0.2) (layer F.Cu) (net 44))
-  (segment (start 270.157535 106.023235) (end 272.757535 106.023235) (width 0.2) (layer F.Cu) (net 44))
-  (segment (start 272.834289 106.099989) (end 279.334289 106.099989) (width 0.2) (layer F.Cu) (net 44))
-  (segment (start 284.401068 111.166768) (end 284.423766 111.166768) (width 0.2) (layer F.Cu) (net 44))
   (segment (start 290.944287 114.400011) (end 290.94431 114.399988) (width 0.2) (layer F.Cu) (net 44))
-  (segment (start 272.757535 106.023235) (end 272.834289 106.099989) (width 0.2) (layer F.Cu) (net 44))
-  (segment (start 263.265 73.495) (end 269.599989 79.829989) (width 0.2) (layer F.Cu) (net 44))
+  (segment (start 290.94431 114.399988) (end 292.25569 114.399988) (width 0.2) (layer F.Cu) (net 44))
   (segment (start 293.1 114.9) (end 293.1 115.7) (width 0.2) (layer F.Cu) (net 44))
-  (segment (start 269.599989 105.465689) (end 270.157535 106.023235) (width 0.2) (layer F.Cu) (net 44))
-  (segment (start 269.599989 79.829989) (end 269.599989 105.465689) (width 0.2) (layer F.Cu) (net 44))
+  (segment (start 292.255713 114.400011) (end 292.600011 114.400011) (width 0.2) (layer F.Cu) (net 44))
+  (segment (start 272.965605 106.099915) (end 272.96568 106.09999) (width 0.2) (layer F.Cu) (net 44))
+  (segment (start 292.600011 114.400011) (end 293.1 114.9) (width 0.2) (layer F.Cu) (net 44))
+  (segment (start 272.96568 106.09999) (end 279.334289 106.09999) (width 0.2) (layer F.Cu) (net 44))
+  (segment (start 270.234214 106.099914) (end 272.965605 106.099915) (width 0.2) (layer F.Cu) (net 44))
   (segment (start 287.657009 114.400011) (end 290.944287 114.400011) (width 0.2) (layer F.Cu) (net 44))
+  (segment (start 279.334289 106.09999) (end 284.401068 111.166768) (width 0.2) (layer F.Cu) (net 44))
+  (segment (start 269.599989 105.465689) (end 270.234214 106.099914) (width 0.2) (layer F.Cu) (net 44))
+  (segment (start 269.599989 79.829989) (end 269.599989 105.465689) (width 0.2) (layer F.Cu) (net 44))
+  (segment (start 292.25569 114.399988) (end 292.255713 114.400011) (width 0.2) (layer F.Cu) (net 44))
+  (segment (start 263.265 73.495) (end 269.599989 79.829989) (width 0.2) (layer F.Cu) (net 44))
+  (segment (start 284.401068 111.166768) (end 284.423766 111.166768) (width 0.2) (layer F.Cu) (net 44))
   (segment (start 278.837222 107.300022) (end 283.904001 112.366801) (width 0.2) (layer F.Cu) (net 45))
   (segment (start 250.599989 84.642489) (end 250.599989 106.73422) (width 0.2) (layer F.Cu) (net 45))
@@
   (segment (start 264.389999 93.669999) (end 263.265 92.545) (width 0.2) (layer F.Cu) (net 51))
   (segment (start 269.199978 98.479978) (end 264.389999 93.669999) (width 0.2) (layer F.Cu) (net 51))
-  (segment (start 269.199978 105.699978) (end 269.199978 98.479978) (width 0.2) (layer F.Cu) (net 51))
+  (segment (start 269.199978 105.699978) (end 269.199978 98.479978) (width 0.2) (layer F.Cu) (net 51) (status 40000))
   (segment (start 269.999923 106.499923) (end 269.199978 105.699978) (width 0.2) (layer F.Cu) (net 51))
   (segment (start 272.799917 106.499924) (end 269.999923 106.499923) (width 0.2) (layer F.Cu) (net 51))

Commit message: Delete regulator
Parts:
- removed C10, C7, C8, C9: 1uF, Capacitor_SMD:C_0603_1608Metric_Pad1.05x0.95mm_HandSolder
- removed D1, D2, D3, D4: D_Small, Diode_SMD:D_SOD-123
- removed R1, R2: R_Small, Resistor_SMD:R_0603_1608Metric_Pad1.05x0.95mm_HandSolder
- removed U10, U9: STLQ015M33R, TO_SOT_Packages_SMD:SOT-23-5
Connections:
- J1 pad 4: Net-(D2-Pad2) -> VCC
- J2 pad 1: Net-(D1-Pad2) -> Net-(J2-Pad1)
- J3 pad 4: Net-(D4-Pad2) -> VAA
- J4 pad 1: Net-(D3-Pad2) -> Net-(J4-Pad1)
- SW1 pad 2: /VCC_BAT -> VCC
- SW1 pad 3: Net-(D1-Pad1) -> Net-(J2-Pad1)
- SW2 pad 2: Net-(D3-Pad1) -> VAA
- SW2 pad 3: /VCC_BAT_R -> Net-(J4-Pad1)
Routing:
- net /VCC_BAT: track 24.6 -> 0.00 mm, vias 1 -> 0
- net /VCC_BAT_R: track 23.8 -> 0.00 mm, vias 1 -> 0
- net VCC: track 24.3 -> 37.1 mm, vias 2 -> 1
- net Net-(D3-Pad2): track 12.5 -> 0.00 mm
- net Net-(J4-Pad1): track 0.00 -> 11.9 mm
- net VAA: track 25.8 -> 36.4 mm, vias 2 -> 1
- net Net-(D1-Pad2): track 10.5 -> 0.00 mm
- net Net-(D1-Pad1): track 9.75 -> 0.00 mm
- net GND: track 28.0 -> 18.3 mm, vias 6 -> 4
- net GNDA: track 26.7 -> 17.9 mm, vias 5 -> 4
- net Net-(J2-Pad1): track 0.00 -> 8.36 mm
- net Net-(D3-Pad1): track 7.20 -> 0.00 mm
- net Net-(D4-Pad2): track 3.90 -> 0.00 mm
- net Net-(D2-Pad2): track 3.90 -> 0.00 mm
- net Net-(SW4-Pad1): track 48.6 -> 46.5 mm
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
Commit message: Add DFU button
Parts:
- added J5: Conn_01x01, locallib:breakout-pad, B.Cu at (67.1, 125.3)
- added J6: Conn_01x01, locallib:breakout-pad, B.Cu at (310.1, 125.3)
- turned SW3 to 0 degrees
Connections:
- SW3 pad 1: Net-(SW3-Pad1) -> GND
- SW3 pad 2: GND -> Net-(SW3-Pad2)
- SW4 pad 1: Net-(SW4-Pad1) -> GNDA
- SW4 pad 2: GNDA -> Net-(SW4-Pad2)
- U1 pad 24: Net-(U1-Pad24) -> Net-(SW3-Pad2)
- U1 pad 7: Net-(SW3-Pad1) -> Net-(J5-Pad1)
- U5 pad 24: Net-(U5-Pad24) -> Net-(SW4-Pad2)
- U5 pad 7: Net-(SW4-Pad1) -> Net-(J6-Pad1)
Routing:
- net Net-(SW4-Pad1): track 46.5 -> 0.00 mm, vias 2 -> 0
- net Net-(SW3-Pad2): track 0.00 -> 33.2 mm, vias 0 -> 2
- net Net-(SW3-Pad1): track 29.5 -> 0.00 mm, vias 2 -> 0
- net Net-(SW4-Pad2): track 0.00 -> 29.4 mm, vias 0 -> 2
- net Net-(J6-Pad1): track 0.00 -> 28.5 mm, vias 0 -> 3
- net Net-(J5-Pad1): track 0.00 -> 17.0 mm, vias 0 -> 1
- net VAA: track 36.4 -> 38.9 mm
- net /L20: track 113.0 -> 111.6 mm
- net /L13: track 131.4 -> 130.0 mm
- net /R14: track 34.3 -> 32.9 mm
- net /R7: track 52.7 -> 51.3 mm
- net VCC: track 37.1 -> 37.8 mm
Other:
- board text added: "RESET"

Commit message: Change matrix wiring
Connections:
- K1 pad 1: GND -> /ROW
- K10 pad 1: GND -> /ROW
- K11 pad 1: GND -> /ROW
- K12 pad 1: GND -> /ROW
- K13 pad 1: GND -> /ROW
- K14 pad 1: GND -> /ROW
- K15 pad 1: GND -> /ROW
- K16 pad 1: GND -> /ROW
- K17 pad 1: GND -> /ROW
- K18 pad 1: GND -> /ROW
- K19 pad 1: GND -> /ROW
- K2 pad 1: GND -> /ROW
- K20 pad 1: GND -> /ROW
- K21 pad 1: GND -> /ROW
- K22 pad 1: GND -> /ROW
- K23 pad 1: GND -> /ROW
- K24 pad 1: GND -> /ROW
- K25 pad 1: GNDA -> /ROW_R
- K26 pad 1: GNDA -> /ROW_R
- K27 pad 1: GNDA -> /ROW_R
- K28 pad 1: GNDA -> /ROW_R
- K29 pad 1: GNDA -> /ROW_R
- K3 pad 1: GND -> /ROW
- K30 pad 1: GNDA -> /ROW_R
- K31 pad 1: GNDA -> /ROW_R
- K32 pad 1: GNDA -> /ROW_R
- K33 pad 1: GNDA -> /ROW_R
- K34 pad 1: GNDA -> /ROW_R
- K35 pad 1: GNDA -> /ROW_R
- K36 pad 1: GNDA -> /ROW_R
- K37 pad 1: GNDA -> /ROW_R
- K38 pad 1: GNDA -> /ROW_R
- K39 pad 1: GNDA -> /ROW_R
- K4 pad 1: GND -> /ROW
- K40 pad 1: GNDA -> /ROW_R
- K41 pad 1: GNDA -> /ROW_R
- K42 pad 1: GNDA -> /ROW_R
- K43 pad 1: GNDA -> /ROW_R
- K44 pad 1: GNDA -> /ROW_R
- K45 pad 1: GNDA -> /ROW_R
- K46 pad 1: GNDA -> /ROW_R
- K47 pad 1: GNDA -> /ROW_R
- K48 pad 1: GNDA -> /ROW_R
- K5 pad 1: GND -> /ROW
- K6 pad 1: GND -> /ROW
- K7 pad 1: GND -> /ROW
- K8 pad 1: GND -> /ROW
- K9 pad 1: GND -> /ROW
- U1 pad 25: Net-(U1-Pad25) -> /ROW
- U5 pad 34: Net-(U5-Pad34) -> /ROW_R
Routing:
- net /ROW_R: track 0.00 -> 505.2 mm, vias 0 -> 1
- net /ROW: track 0.00 -> 498.2 mm, vias 0 -> 1
- net GNDA: track 17.9 -> 25.4 mm
Other:
- board text added: "Caravelle-BLE PCB v2.1 by SatT"
- board text added: "OFF"
- board text added: "ON"
- board text removed: "Caravelle-BLE PCB v2.0 by SatT"

Commit message: Fix capacitor location & refine wiring
Parts:
- moved C4 3.83 mm to (303.2, 115.1), turned to 180 degrees
- moved C1 1.87 mm to (88.0, 113.3)
Routing:
- net Net-(J6-Pad1): track 28.5 -> 20.7 mm
- net VCC: track 37.8 -> 42.0 mm
- net GNDA: track 25.4 -> 28.0 mm
- net VAA: track 39.2 -> 37.3 mm
- net GND: track 18.3 -> 20.2 mm
- net /R14: track 32.9 -> 34.2 mm
- net /R1: track 69.7 -> 71.0 mm
- net /R8: track 41.0 -> 42.3 mm
- net /R2: track 61.0 -> 62.3 mm
- net /R15: track 21.0 -> 22.3 mm
- net /R7: track 51.3 -> 52.6 mm
Other:
- board text added: "Caravelle-BLE PCB v2.2 by SatT"
- board text removed: "Caravelle-BLE PCB v2.1 by SatT"
