File: caravelle.kicad_pcb (KiCad board)
At the start: 2 copper layers, 277.4 x 94.1 mm, 71 parts, among them J1 Conn_01x04, J2 Conn_01x02_Female, J3 Conn_01x04, J4 Conn_01x02_Female, J5 Conn_01x01, J6 Conn_01x01, K1 keyboard_parts_KEYSW, K10 keyboard_parts_KEYSW, K11 keyboard_parts_KEYSW, K12 keyboard_parts_KEYSW, K13 keyboard_parts_KEYSW, K14 keyboard_parts_KEYSW, K15 keyboard_parts_KEYSW, K16 keyboard_parts_KEYSW, K17 keyboard_parts_KEYSW, K18 keyboard_parts_KEYSW, K19 keyboard_parts_KEYSW, K2 keyboard_parts_KEYSW, K20 keyboard_parts_KEYSW, K21 keyboard_parts_KEYSW, K22 keyboard_parts_KEYSW, K23 keyboard_parts_KEYSW, K24 keyboard_parts_KEYSW, K25 keyboard_parts_KEYSW, K26 keyboard_parts_KEYSW, K27 keyboard_parts_KEYSW, K28 keyboard_parts_KEYSW, K29 keyboard_parts_KEYSW, K3 keyboard_parts_KEYSW, K30 keyboard_parts_KEYSW, K31 keyboard_parts_KEYSW, K32 keyboard_parts_KEYSW, K33 keyboard_parts_KEYSW, K34 keyboard_parts_KEYSW, K35 keyboard_parts_KEYSW, K36 keyboard_parts_KEYSW, K37 keyboard_parts_KEYSW, K38 keyboard_parts_KEYSW, K39 keyboard_parts_KEYSW, K4 keyboard_parts_KEYSW, K40 keyboard_parts_KEYSW, K41 keyboard_parts_KEYSW, K42 keyboard_parts_KEYSW, K43 keyboard_parts_KEYSW, K44 keyboard_parts_KEYSW, K45 keyboard_parts_KEYSW, K46 keyboard_parts_KEYSW, K47 keyboard_parts_KEYSW, K48 keyboard_parts_KEYSW, K5 keyboard_parts_KEYSW, K6 keyboard_parts_KEYSW, K7 keyboard_parts_KEYSW, K8 keyboard_parts_KEYSW, K9 keyboard_parts_KEYSW, SW1 SW_SPDT, SW2 SW_SPDT, SW3 RESET_SW, SW4 RESET_SW, U1 BL652_LEFT, U11 logo1, U12 logo2, U13 logo1, U2 hole, U3 hole, U4 hole, U5 BL652_RIGHT, U6 hole, U7 hole, U8 hole

Commit message: Add edge rails for PCBA
Parts:
- added U10: hole, Fiducial:Fiducial_1mm_Mask3mm, F.Cu at (65.0, 42.0)
- added U14: hole, Fiducial:Fiducial_0.75mm_Mask2.25mm, F.Cu at (65.0, 152.0)
- added U15: hole, MountingHole:MountingHole_4mm, F.Cu at (55.0, 42.0)
- added U16: hole, MountingHole:MountingHole_4mm, F.Cu at (322.4, 152.0)
- added U17: hole, MountingHole:MountingHole_4mm, F.Cu at (55.0, 152.0)
- added U18: hole, MountingHole:MountingHole_4mm, F.Cu at (322.4, 42.0)
- added U19: hole, random-keyboard-parts:breakaway-mousebites, F.Cu at (64.0, 130.1)
- added U20: hole, random-keyboard-parts:breakaway-mousebites, F.Cu at (142.9, 133.9)
- added U21: hole, random-keyboard-parts:breakaway-mousebites, F.Cu at (234.5, 134.0)
- added U22: hole, random-keyboard-parts:breakaway-mousebites, F.Cu at (313.4, 130.0)
- added U23: hole, Fiducial:Fiducial_0.75mm_Mask2.25mm, F.Cu at (317.4, 42.0)
- added U9: hole, Fiducial:Fiducial_1mm_Mask3mm, F.Cu at (317.4, 152.0)
- moved U8 134.8 mm to (313.4, 59.3), turned to 180 degrees
- moved U2 121.2 mm to (64.0, 59.3), turned to 180 degrees
- moved U3 100.2 mm to (98.2, 53.3), turned to 180 degrees
- moved U7 100.2 mm to (279.2, 53.3), turned to 180 degrees
- moved U4 66.4 mm to (173.8, 66.4), turned to 180 degrees
- moved U6 16.2 mm to (203.6, 66.4), turned to 180 degrees
Connections:
- SW1 pad 1: Net-(SW1-Pad1) -> (no net)
- SW2 pad 1: Net-(SW2-Pad1) -> (no net)
- U1 pad 14: Net-(U1-Pad14) -> (no net)
- U1 pad 15: Net-(U1-Pad15) -> (no net)
- U1 pad 2: Net-(U1-Pad2) -> (no net)
- U1 pad 3: Net-(U1-Pad3) -> (no net)
- U1 pad 4: Net-(U1-Pad4) -> (no net)
- U5 pad 14: Net-(U5-Pad14) -> (no net)
- U5 pad 15: Net-(U5-Pad15) -> (no net)
- U5 pad 35: Net-(U5-Pad35) -> (no net)
- U5 pad 37: Net-(U5-Pad37) -> (no net)
- U5 pad 38: Net-(U5-Pad38) -> (no net)
Other:
- board size 277.4 x 94.1 mm -> 277.4 x 120 mm

Commit message: Clean up Fab
Parts:
- U10, U14, U23, U9: value hole -> fiducial
- U15, U16, U17, U18: footprint MountingHole:MountingHole_4mm -> locallib:MountingHole_4mm

Commit message: Furthermore cleanup
Parts:
- C1, C4: footprint Capacitor_SMD:C_0603_1608Metric_Pad1.05x0.95mm_HandSolder -> Capacitor_SMD:C_0603_1608Metric
- U11, U13: value logo1 -> hole

Commit message: Add Kailh hotswap footprint
Parts:
- C1, C4: footprint Capacitor_SMD:C_0603_1608Metric -> Capacitor_SMD:C_0603_1608Metric_Pad1.05x0.95mm_HandSolder
- K1, K10, K11, K12, K13, K14, K15, K16, K17, K18, K19, K2, K20, K23, K25, K26, K27, K28, K29, K3, K30, K31, K32, K33, K34, K35, K36, K37, K38, K39, K4, K40, K41, K42, K43, K44, K47, K5, K6, K7, K8, K9: footprint MX_Only:MXOnly-1U-NoLED -> MX_Only:MXOnly-1U-Hotswap-Antishear
- K21, K22, K45, K46: footprint MX_Only:MXOnly-1.25U-NoLED -> locallib:MXOnly-1.25U-Hotswap-Antishear
- K24, K48: footprint MX_Only:MXOnly-1.5U-NoLED -> locallib:MXOnly-1.5U-Hotswap-Antishear
- U11, U13: value hole -> logo1
- U15, U16, U17, U18: footprint locallib:MountingHole_4mm -> MountingHole:MountingHole_4mm
